Commit message: updated URDF

File: urdf/ur_table.urdf.xacro (robot description, xacro)
@@ -51,9 +51,10 @@
    <!-- create link fixed to the "world" -->
    <link name="world" />
+   <!--
    <link name="table">
      <visual>
        <origin xyz="0 0 0" rpy="0 0 0"/>
        <geometry>
-         <mesh filename="package://magician_demo/resources/mesh/tavolo.stl" scale="0.001 0.001 0.001"/>
+         <mesh filename="package://magician_ur/resources/mesh/tavolo.stl" scale="0.001 0.001 0.001"/>
        </geometry>
        <material name="white">
@@ -64,5 +65,5 @@
        <origin xyz="0 0 0" rpy="0 0 0"/>
        <geometry>
-         <mesh filename="package://magician_demo/resources/mesh/tavolo.stl" scale="0.001 0.001 0.001"/>
+         <mesh filename="package://magician_ur/resources/mesh/tavolo.stl" scale="0.001 0.001 0.001"/>
        </geometry>
      </collision>
@@ -73,4 +74,5 @@
      <child link="table" />
    </joint>
+   -->
    <!-- arm -->
    <xacro:ur_robot

Commit message: Added bota ft sensor

File: urdf/ur_table.urdf.xacro (robot description, xacro)
@@ -113,4 +113,27 @@
    <origin xyz="0.510 0.340 1.789" rpy="${pi} 0 ${pi}" />          <!-- position robot in the world -->
    </xacro:ur_robot>
+  <xacro:include filename="$(find rokubimini_description)/urdf/BFT_SENS_ECAT_M8.urdf.xacro" />
+    <xacro:BFT_SENS_ECAT_M8 prefix="ft_sensor0" />
+    <joint name="bota_ft_sensor" type="fixed">
+      <parent link="ft_frame" />
+      <child link = "ft_sensor0_mounting" />
+      <origin xyz="0.0 0.0 0.0" rpy="${pi} 0.0 ${pi/2}" />
+    </joint>
+    <link
+      name="probe">
+    </link>
+    <joint name="tip_tool" type="fixed">
+      <parent link="ft_sensor0_wrench" />
+      <child link = "probe" />
+      <origin xyz="0.0 0.0 0.08" rpy="0.0 0.0 0.0" />
+    </joint>
+    <link
+      name="compliance_link">
+    </link>
+    <joint name="tool_to_compliance" type="fixed">
+      <parent link="probe" />
+      <child link = "compliance_link" />
+      <origin xyz="0.0 0.0 0.045" rpy="0.0 0.0 0.0" />
+    </joint>
    <xacro:if value="$(arg sim_gazebo)">
     <!-- Gazebo plugins -->

Commit message: Updated table setup

File: urdf/ur_table.urdf.xacro (robot description, xacro)
@@ -134,5 +134,5 @@
       <parent link="probe" />
       <child link = "compliance_link" />
-      <origin xyz="0.0 0.0 0.045" rpy="0.0 0.0 0.0" />
+      <origin xyz="0.0 0.0 0.0" rpy="0.0 0.0 0.0" />
     </joint>
    <xacro:if value="$(arg sim_gazebo)">
